File: FSAE_Analog_to_CAN_Converter/FSAE_Analog_to_CAN_Converter.kicad_sch (KiCad schematic)
At the start: 32 parts, among them J1 Conn_01x07_Pin, J2 Conn_01x02_Pin, J3 Conn_01x05, U1 AP63205WU, U2 LT1962-3.3, U3 STM32F103RCTx, U4 MCP2562-E-MF, Y1 8MHz

Commit message: production files and no DRC errors
Parts:
- removed U4: MCP2562-E-MF, Package_DFN_QFN:DFN-8-1EP_3x3mm_P0.65mm_EP1.55x2.4mm, symbol Interface_CAN_LIN:MCP2562-E-MF
- added U5: MCP2562-E-SN, Package_SO:SOIC-8_3.9x4.9mm_P1.27mm, symbol Interface_CAN_LIN:MCP2562-E-SN
- R1: footprint Resistor_SMD:R_0201_0603Metric_Pad0.64x0.40mm_HandSolder -> Resistor_SMD:R_0805_2012Metric_Pad1.20x1.40mm_HandSolder
Connections:
- net +3.3V: now also U5.5 (Vio)
- net +5V: now also U5.3 (VDD)
- net CAN_OUT_N: now also U5.6 (CANL)
- net CAN_OUT_P: now also U5.7 (CANH)
- net CAN_RX: now also U5.4 (RXD)
- net CAN_TX: now also U5.1 (TXD)
- net GND: now also U5.2 (VSS), U5.8 (STBY)
Changed lines of the file:
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@@
 	)
 	(junction
-		(at 243.84 132.08)
-		(diameter 0)
-		(color 0 0 0 0)
-	)
-	(junction
 		(at 257.81 121.92)
 		(diameter 0)
@@
 	)
 	(junction
+		(at 243.84 132.08)
+		(diameter 0)
+		(color 0 0 0 0)
+	)
+	(junction
 		(at 257.81 116.84)
 		(diameter 0)
@@
 	)
 	(junction
-		(at 228.6 124.46)
-		(diameter 0)
-		(color 0 0 0 0)
-	)
-	(junction
 		(at 153.67 33.02)
 		(diameter 0)
@@
 	(wire
 		(pts
-			(xy 241.3 132.08) (xy 241.3 129.54)
-		)
-		(stroke
-			(width 0)
-			(type default)
-		)
-	)
-	(wire
-		(pts
 			(xy 87.63 52.07) (xy 87.63 54.61)
 		)
@@
 	(wire
 		(pts
-			(xy 228.6 135.89) (xy 228.6 124.46)
-		)
-		(stroke
-			(width 0)
-			(type default)
-		)
-	)
-	(wire
-		(pts
-			(xy 228.6 124.46) (xy 231.14 124.46)
-		)
-		(stroke
-			(width 0)
-			(type default)
-		)
-	)
-	(wire
-		(pts
 			(xy 257.81 124.46) (xy 257.81 121.92)
 		)
@@
 	(wire
 		(pts
-			(xy 243.84 132.08) (xy 241.3 132.08)
+			(xy 186.69 76.2) (xy 186.69 78.74)
 		)
 		(stroke
@@
 	(wire
 		(pts
-			(xy 186.69 76.2) (xy 186.69 78.74)
+			(xy 76.2 46.99) (xy 77.47 46.99)
 		)
 		(stroke
@@
 	(wire
 		(pts
-			(xy 76.2 46.99) (xy 77.47 46.99)
+			(xy 269.24 43.18) (xy 281.94 43.18)
 		)
 		(stroke
@@
 	(wire
 		(pts
-			(xy 269.24 43.18) (xy 281.94 43.18)
+			(xy 295.91 85.09) (xy 295.91 87.63)
 		)
 		(stroke
@@
 	(wire
 		(pts
-			(xy 295.91 85.09) (xy 295.91 87.63)
+			(xy 124.46 48.26) (xy 124.46 55.88)
 		)
 		(stroke
@@
 	(wire
 		(pts
-			(xy 124.46 48.26) (xy 124.46 55.88)
+			(xy 231.14 124.46) (xy 231.14 132.08)
 		)
 		(stroke
@@
 	(wire
 		(pts
+			(xy 231.14 132.08) (xy 243.84 132.08)
+		)
+		(stroke
+			(width 0)
+			(type default)
+		)
+	)
+	(wire
+		(pts
 			(xy 218.44 43.18) (xy 231.14 43.18)
 		)
@@
 	(wire
 		(pts
-			(xy 228.6 124.46) (xy 228.6 121.92)
+			(xy 228.6 121.92) (xy 228.6 135.89)
 		)
 		(stroke
@@
 	)
 	(symbol
+		(lib_id "Interface_CAN_LIN:MCP2562-E-SN")
+		(at 243.84 119.38 0)
+		(unit 1)
+		(body_style 1)
+		(exclude_from_sim no)
+		(in_bom yes)
+		(on_board yes)
+		(in_pos_files yes)
+		(dnp no)
+		(fields_autoplaced yes)
+		(property "Reference" "U5"
+			(at 245.9833 106.68 0)
+			(show_name no)
+			(do_not_autoplace no)
+			(effects
+				(font
+					(size 1.27 1.27)
+				)
+				(justify left)
+			)
+		)
+		(property "Value" "MCP2562-E-SN"
+			(at 245.9833 109.22 0)
+			(show_name no)
+			(do_not_autoplace no)
+			(effects
+				(font
+					(size 1.27 1.27)
+				)
+				(justify left)
+			)
+		)
+		(property "Footprint" "Package_SO:SOIC-8_3.9x4.9mm_P1.27mm"
+			(at 243.84 132.08 0)
+			(hide yes)
+			(show_name no)
+			(do_not_autoplace no)
+			(effects
+				(font
+					(size 1.27 1.27)
+					(italic yes)
+				)
+			)
+		)
+		(property "Datasheet" "http://ww1.microchip.com/downloads/en/DeviceDoc/25167A.pdf"
+			(at 243.84 119.38 0)
+			(hide yes)
+			(show_name no)
+			(do_not_autoplace no)
+			(effects
+				(font
+					(size 1.27 1.27)
+				)
+			)
+		)
+		(property "Description" "High-Speed CAN Transceiver, 1Mbps, 5V supply, Vio pin, -40C to +125C, SOIC-8"
+			(at 243.84 119.38 0)
+			(hide yes)
+			(show_name no)
+			(do_not_autoplace no)
+			(effects
+				(font
+					(size 1.27 1.27)
+				)
+			)
+		)
+		(pin "5"
+		)
+		(pin "6"
+		)
+		(pin "2"
+		)
+		(pin "7"
+		)
+		(pin "4"
+		)
+		(pin "3"
+		)
+		(pin "8"
+		)
+		(pin "1"
+		)
+		(instances
+			(project "FSAE_Analog_to_CAN_Converter"
+				(path "/99368ba7-2b2d-46bc-b71f-42c7765e3ed8"
+					(reference "U5")
+					(unit 1)
+				)
+			)
+		)
+	)
+	(symbol
 		(lib_id "MCU_ST_STM32F1:STM32F103RCTx")
 		(at 189.23 127 0)
@@
 			)
 		)
-		(property "Footprint" "Resistor_SMD:R_0201_0603Metric_Pad0.64x0.40mm_HandSolder"
+		(property "Footprint" "Resistor_SMD:R_0805_2012Metric_Pad1.20x1.40mm_HandSolder"
 			(at 160.528 97.79 90)
 			(hide yes)
@@
 					(unit 1)
 				)
-			)
-		)
-	)
-	(symbol
-		(lib_id "Interface_CAN_LIN:MCP2562-E-MF")
-		(at 243.84 119.38 0)
-		(unit 1)
-		(body_style 1)
-		(exclude_from_sim no)
-		(in_bom yes)
-		(on_board yes)
-		(in_pos_files yes)
-		(dnp no)
-		(fields_autoplaced yes)
-		(property "Reference" "U4"
-			(at 245.9833 106.68 0)
-			(show_name no)
-			(do_not_autoplace no)
-			(effects
-				(font
-					(size 1.27 1.27)
-				)
-				(justify left)
-			)
-		)
-		(property "Value" "MCP2562-E-MF"
-			(at 245.9833 109.22 0)
-			(show_name no)
-			(do_not_autoplace no)
-			(effects
-				(font
-					(size 1.27 1.27)
-				)
-				(justify left)
-			)
-		)
-		(property "Footprint" "Package_DFN_QFN:DFN-8-1EP_3x3mm_P0.65mm_EP1.55x2.4mm"
-			(at 243.84 132.08 0)
-			(hide yes)
-			(show_name no)
-			(do_not_autoplace no)
-			(effects
-				(font
-					(size 1.27 1.27)
-					(italic yes)
-				)
-			)
-		)
-		(property "Datasheet" "http://ww1.microchip.com/downloads/en/DeviceDoc/25167A.pdf"
-			(at 243.84 119.38 0)
-			(hide yes)
-			(show_name no)
-			(do_not_autoplace no)
-			(effects
-				(font
-					(size 1.27 1.27)
-				)
-			)
-		)
-		(property "Description" "High-Speed CAN Transceiver, 1Mbps, 5V supply, Vio pin, -40C to +125C, DFN-8"
-			(at 243.84 119.38 0)
-			(hide yes)
-			(show_name no)
-			(do_not_autoplace no)
-			(effects
-				(font
-					(size 1.27 1.27)
-				)
-			)
-		)
-		(pin "7"
-		)
-		(pin "3"
-		)
-		(pin "4"
-		)
-		(pin "6"
-		)
-		(pin "1"
-		)
-		(pin "2"
-		)
-		(pin "5"
-		)
-		(pin "9"
-		)
-		(pin "8"
-		)
-		(instances
-			(project "FSAE_Analog_to_CAN_Converter"
-				(path "/99368ba7-2b2d-46bc-b71f-42c7765e3ed8"
-					(reference "U4")
-					(unit 1)
-				)
