File: FSAE_Analog_to_CAN_Converter/FSAE_Analog_to_CAN_Converter.kicad_pcb (KiCad board)
At the start: 4 copper layers, 55 x 45 mm, 32 parts, among them J1 Conn_01x07_Pin, J2 Conn_01x02_Pin, J3 Conn_01x05, U1 AP63205WU, U2 LT1962-3.3, U3 STM32F103RCTx, U5 MCP2562-E-SN, Y1 8MHz

Commit message: minor stuff
Routing:
- net /SWCLK: track 26.7 -> 23.5 mm
- net +5V: track 44.0 -> 42.7 mm, vias 8 -> 7
Other:
- board size 55 x 45 mm -> 60 x 44.2 mm
- board text added: "+12V"
- board text added: "AIN 1"
- board text added: "AIN 2"
- board text added: "AIN 3"
- board text added: "AIN 4"
- board text added: "AIN 5"
- board text added: "FSAE Analog to CAN Converter Rev 1."
Changed lines of the file:
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@@
 	)
 	(gr_arc
-		(start 53 33)
-		(mid 55.050253 28.050253)
-		(end 60 26)
+		(start 48 36.75)
+		(mid 50.928932 29.678932)
+		(end 58 26.75)
 		(stroke
 			(width 0.05)
@@
 	)
 	(gr_line
-		(start 53 64)
-		(end 53 33)
+		(start 48 61)
+		(end 48 36.75)
 		(stroke
 			(width 0.05)
@@
 	)
 	(gr_line
-		(start 60 26)
-		(end 92 26)
+		(start 58 26.75)
+		(end 98 26.75)
 		(stroke
 			(width 0.05)
@@
 	)
 	(gr_arc
-		(start 60 71)
-		(mid 55.050253 68.949747)
-		(end 53 64)
+		(start 58 71)
+		(mid 50.928932 68.071068)
+		(end 48 61)
 		(stroke
 			(width 0.05)
@@
 	)
 	(gr_arc
-		(start 92 26)
-		(mid 96.949747 28.050253)
-		(end 99 33)
+		(start 98 26.75)
+		(mid 105.071068 29.678932)
+		(end 108 36.75)
 		(stroke
 			(width 0.05)
@@
 	)
 	(gr_line
-		(start 99 33)
-		(end 99 38)
+		(start 98 71)
+		(end 58 71)
 		(stroke
 			(width 0.05)
@@
 	)
 	(gr_line
-		(start 101 71)
-		(end 60 71)
+		(start 108 36.75)
+		(end 108 61)
 		(stroke
 			(width 0.05)
@@
 	)
 	(gr_arc
-		(start 106 45)
-		(mid 101.050253 42.949747)
-		(end 99 38)
+		(start 108 61)
+		(mid 105.071068 68.071068)
+		(end 98 71)
 		(stroke
 			(width 0.05)
@@
 		(layer "Edge.Cuts")
 	)
-	(gr_arc
-		(start 106 45)
-		(mid 107.414214 45.585786)
-		(end 108 47)
-		(stroke
-			(width 0.05)
-			(type default)
-		)
-		(layer "Edge.Cuts")
-	)
-	(gr_line
-		(start 108 47)
-		(end 108 64)
-		(stroke
-			(width 0.05)
-			(type default)
-		)
-		(layer "Edge.Cuts")
-	)
-	(gr_arc
-		(start 108 64)
-		(mid 105.949747 68.949747)
-		(end 101 71)
-		(stroke
-			(width 0.05)
-			(type default)
-		)
-		(layer "Edge.Cuts")
+	(gr_text "AIN 5\n"
+		(at 50 56.8 0)
+		(layer "F.SilkS")
+		(effects
+			(font
+				(size 1 1)
+				(thickness 0.15)
+			)
+			(justify left bottom)
+		)
+	)
+	(gr_text "+12V"
+		(at 50.2 39 0)
+		(layer "F.SilkS")
+		(effects
+			(font
+				(size 1 1)
+				(thickness 0.15)
+			)
+			(justify left bottom)
+		)
+	)
+	(gr_text "AIN 1\n"
+		(at 50.2 44.8 0)
+		(layer "F.SilkS")
+		(effects
+			(font
+				(size 1 1)
+				(thickness 0.15)
+			)
+			(justify left bottom)
+		)
+	)
+	(gr_text "AIN 2\n"
+		(at 50.2 47.8 0)
+		(layer "F.SilkS")
+		(effects
+			(font
+				(size 1 1)
+				(thickness 0.15)
+			)
+			(justify left bottom)
+		)
+	)
+	(gr_text "AIN 3\n"
+		(at 50.2 50.8 0)
+		(layer "F.SilkS")
+		(effects
+			(font
+				(size 1 1)
+				(thickness 0.15)
+			)
+			(justify left bottom)
+		)
+	)
+	(gr_text "AIN 4\n"
+		(at 50.2 53.8 0)
+		(layer "F.SilkS")
+		(effects
+			(font
+				(size 1 1)
+				(thickness 0.15)
+			)
+			(justify left bottom)
+		)
+	)
+	(gr_text "GND\n"
+		(at 51.2 42 0)
+		(layer "F.SilkS")
+		(effects
+			(font
+				(size 1 1)
+				(thickness 0.15)
+			)
+			(justify left bottom)
+		)
+	)
+	(gr_text "FSAE Analog to CAN Converter Rev 1.\n"
+		(at 57.75 70 0)
+		(layer "F.SilkS")
+		(effects
+			(font
+				(size 1 1)
+				(thickness 0.15)
+			)
+			(justify left bottom)
+		)
 	)
 	(gr_text "CANH\n"
@@
 	)
 	(segment
-		(start 90.1 56.8375)
-		(end 90.1 57.8)
-		(width 0.2)
-		(layer "F.Cu")
-		(net "+5V")
-	)
-	(segment
 		(start 82.3859 36.9084)
 		(end 82.1675 36.69)
@@
 	)
 	(segment
-		(start 90.1 57.8)
-		(end 90.3 58)
-		(width 0.2)
-		(layer "F.Cu")
-		(net "+5V")
-	)
-	(segment
 		(start 87.2744 34.7726)
 		(end 87.503 34.7726)
@@
 	(via
 		(at 87.9348 40.3606)
-		(size 0.6)
-		(drill 0.3)
-		(layers "F.Cu" "B.Cu")
-		(net "+5V")
-	)
-	(via
-		(at 90.3 58)
 		(size 0.6)
 		(drill 0.3)
@@
 	)
 	(segment
-		(start 85.25 51.75)
-		(end 84.4 52.6)
+		(start 86.075 51.75)
+		(end 85.05 51.75)
 		(width 0.2)
 		(layer "F.Cu")
@@
 	)
 	(segment
-		(start 86.075 51.75)
-		(end 85.25 51.75)
+		(start 84.4 52.4)
+		(end 84.4 58.4)
 		(width 0.2)
 		(layer "F.Cu")
@@
 	)
 	(segment
-		(start 86.9 61.1)
-		(end 89.62 61.1)
+		(start 89.72 61.2)
+		(end 91.92 63.4)
 		(width 0.2)
 		(layer "F.Cu")
@@
 	)
 	(segment
-		(start 84.4 52.6)
-		(end 84.4 58.6)
+		(start 85.05 51.75)
+		(end 84.4 52.4)
 		(width 0.2)
 		(layer "F.Cu")
@@
 	)
 	(segment
-		(start 84.4 58.6)
-		(end 86.9 61.1)
+		(start 84.4 58.4)
+		(end 87.2 61.2)
 		(width 0.2)
 		(layer "F.Cu")
@@
 	)
 	(segment
-		(start 89.62 61.1)
-		(end 91.92 63.4)
+		(start 87.2 61.2)
+		(end 89.72 61.2)
 		(width 0.2)
 		(layer "F.Cu")
@@
 	)
 	(segment
-		(start 84.15 47.95)
-		(end 84.9 47.2)
+		(start 84.15 47.65)
+		(end 84.8 47)
 		(width 0.2)
 		(layer "F.Cu")
@@
 	(segment
 		(start 84.15 48.825)
-		(end 84.15 47.95)
+		(end 84.15 47.65)
 		(width 0.2)
 		(layer "F.Cu")
@@
 	)
 	(via
-		(at 84.9 47.2)
+		(at 84.8 47)
 		(size 0.6)
 		(drill 0.3)
@@
 	)
 	(segment
-		(start 84.9 47.2)
-		(end 90.948529 47.2)
+		(start 84.8 47.148529)
+		(end 93.31 55.658529)
 		(width 0.2)
 		(layer "B.Cu")
@@
 	)
 	(segment
-		(start 96.8875 63.2875)
+		(start 93.31 59.71)
 		(end 97 63.4)
 		(width 0.2)
@@
 	)
 	(segment
-		(start 90.948529 47.2)
-		(end 96.8875 53.138971)
+		(start 84.8 47)
+		(end 84.8 47.148529)
 		(width 0.2)
 		(layer "B.Cu")
@@
 	)
 	(segment
-		(start 96.8875 53.138971)
-		(end 96.8875 63.2875)
+		(start 93.31 55.658529)
+		(end 93.31 59.71)
 		(width 0.2)
 		(layer "B.Cu")
